File: Hardware/Smart_Watch/POWER SUPPLY.kicad_sch (KiCad schematic)
At the start: 20 parts, among them U3 TLV62568DBV, U4 TLV62568DBV

Commit message: add screen
Parts:
- removed TP2, TP3, TP4: ~, TestPoint:TestPoint_Pad_D1.0mm, symbol Connector:TestPoint
