File: Hardware/Smart_Watch/RP2040.kicad_sch (KiCad schematic)
At the start: 37 parts, among them J1 USB_C_Receptacle_USB2.0, SW1 PICO BOOT, SW2 PICO RST, U1 W25Q128JVS, U2 RP2040, Y1 12.000MHZ

Commit message: update layout pcb
Parts:
- removed C11, C12, C4: 100nF, Capacitor_SMD:C_0402_1005Metric, symbol Device:C
- removed D2, D3: LED, LED_SMD:LED_0603_1608Metric, symbol Device:LED
- removed R10, R11, R12, R13, R9: 22R, Resistor_SMD:R_0402_1005Metric, symbol Device:R
- removed R14, R15: 330R, Resistor_SMD:R_0402_1005Metric, symbol Device:R
Connections:
- net FPGA_MISO: no longer names the net of U2.11 (GPIO8)
- net FPGA_MOSI: no longer names the net of U2.14 (GPIO11)
- net FPGA_SDCS: no longer names the net of U2.12 (GPIO9)
- net GP0: no longer names the net of U2.2 (GPIO0)
- net GP1: no longer names the net of U2.3 (GPIO1)
- net GP2: no longer names the net of U2.4 (GPIO2)
- net GP20: no longer names the net of U2.31 (GPIO20)
- net GP21: no longer names the net of U2.32 (GPIO21)
- net GP22: no longer names the net of U2.34 (GPIO22)
- net GP23: no longer names the net of U2.35 (GPIO23)
- net GP3: no longer names the net of U2.5 (GPIO3)
- net GP4: no longer names the net of U2.6 (GPIO4)
- net GP5: no longer names the net of U2.7 (GPIO5)
- net GP6: no longer names the net of U2.8 (GPIO6)
- net GP7: no longer names the net of U2.9 (GPIO7)
- net RXD: no longer names the net of U2.16 (GPIO13)
- net TCK: no longer names the net of U2.29 (GPIO18)
- net TDI: no longer names the net of U2.27 (GPIO16)
- net TDO: no longer names the net of U2.28 (GPIO17)
- net TMS: no longer names the net of U2.30 (GPIO19)
- net TXD: no longer names the net of U2.15 (GPIO12)
- no-connect marks 8 -> 6
Other:
- note removed: "MISO"
- note removed: "MOSI"
- note removed: "RXD"
- note removed: "SCK"
- note removed: "SS"
- note removed: "TXD"

Commit message: add screen
Parts:
- removed C5: 22uF, Capacitor_SMD:C_0603_1608Metric, symbol Device:C
- removed D1: SS34, Diode_SMD:D_SMA, symbol Device:D
Connections:
- net +5V: now also J1.A4 (VBUS), J1.A9 (VBUS), J1.B4 (VBUS), J1.B9 (VBUS)
- net RESET: now reaches U2.18 (GPIO15)
- net DC: now reaches U2.27 (GPIO16)
- net CS: now reaches U2.28 (GPIO17)
- net SCK: now reaches U2.29 (GPIO18)
- net SDI: now reaches U2.30 (GPIO19)
