File: Hardware/Smart_Watch/Screen_TFT.kicad_sch (KiCad schematic)
At the start: 0 parts

Commit message: add screen
Parts:
- added J2: Conn_01x12, Footprint:GC9A01_Extended_FPC, symbol Connector_Generic:Conn_01x12
Connections:
- new net +3.3V: J2.4 (Pin_4)
- new net CS: J2.8 (Pin_8)
- new net DC: J2.7 (Pin_7)
- new net GND: J2.1 (Pin_1), J2.12 (Pin_12), J2.5 (Pin_5), J2.6 (Pin_6)
- new net RESET: J2.11 (Pin_11)
- new net SCK: J2.9 (Pin_9)
- new net SDI: J2.10 (Pin_10)
- no-connect marks 0 -> 2
